File: CanSatPCB/CanSatPCB.kicad_sch (KiCad schematic)
At the start: 0 parts

Commit message: test 1
Parts:
- added U1: ESP32-S3-MINI-1U, RF_Module:ESP32-S2-MINI-1U, symbol RF_Module:ESP32-S3-MINI-1U
Connections:
- new net: U1.1 (GND), U1.2 (GND), U1.42 (GND), U1.43 (GND), U1.46 (GND), U1.47 (GND), U1.48 (GND), U1.49 (GND), U1.50 (GND), U1.51 (GND), U1.52 (GND), U1.53 (GND), U1.54 (GND), U1.55 (GND), U1.56 (GND), U1.57 (GND), U1.58 (GND), U1.59 (GND), U1.60 (GND), U1.61 (GND), U1.62 (GND), U1.63 (GND), U1.64 (GND), U1.65 (GND)
Changed lines of the file:
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@@
 	(generator_version "9.0")
 	(paper "A4")
+	(symbol
+		(lib_id "RF_Module:ESP32-S3-MINI-1U")
+		(at 100.33 54.61 0)
+		(unit 1)
+		(exclude_from_sim no)
+		(in_bom yes)
+		(on_board yes)
+		(dnp no)
+		(fields_autoplaced yes)
+		(property "Reference" "U1"
+			(at 102.4733 21.59 0)
+			(effects
+				(font
+					(size 1.27 1.27)
+				)
+				(justify left)
+			)
+		)
+		(property "Value" "ESP32-S3-MINI-1U"
+			(at 102.4733 24.13 0)
+			(effects
+				(font
+					(size 1.27 1.27)
+				)
+				(justify left)
+			)
+		)
+		(property "Footprint" "RF_Module:ESP32-S2-MINI-1U"
+			(at 116.84 83.82 0)
+			(effects
+				(font
+					(size 1.27 1.27)
+				)
+				(hide yes)
+			)
+		)
+		(property "Datasheet" "https://www.espressif.com/sites/default/files/documentation/esp32-s3-mini-1_mini-1u_datasheet_en.pdf"
+			(at 100.33 13.97 0)
+			(effects
+				(font
+					(size 1.27 1.27)
+				)
+				(hide yes)
+			)
+		)
+		(property "Description" "RF Module, ESP32-S3 SoC, Wi-Fi 802.11b/g/n, Bluetooth, BLE, 32-bit, 3.3V, SMD, external antenna"
+			(at 100.33 11.43 0)
+			(effects
+				(font
+					(size 1.27 1.27)
+				)
+				(hide yes)
+			)
+		)
+		(pin "12"
+		)
+		(pin "5"
+		)
+		(pin "7"
+		)
+		(pin "11"
+		)
+		(pin "6"
+		)
+		(pin "4"
+		)
+		(pin "8"
+		)
+		(pin "9"
+		)
+		(pin "45"
+		)
+		(pin "10"
+		)
+		(pin "13"
+		)
+		(pin "14"
+		)
+		(pin "15"
+		)
+		(pin "16"
+		)
+		(pin "17"
+		)
+		(pin "18"
+		)
+		(pin "19"
+		)
+		(pin "20"
+		)
+		(pin "22"
+		)
+		(pin "3"
+		)
+		(pin "1"
+		)
+		(pin "21"
+		)
+		(pin "2"
+		)
+		(pin "42"
+		)
+		(pin "53"
+		)
+		(pin "23"
+		)
+		(pin "46"
+		)
+		(pin "61"
+		)
+		(pin "58"
+		)
+		(pin "55"
+		)
+		(pin "56"
+		)
+		(pin "63"
+		)
+		(pin "50"
+		)
+		(pin "51"
+		)
+		(pin "64"
+		)
+		(pin "62"
+		)
+		(pin "25"
+		)
+		(pin "32"
+		)
+		(pin "26"
+		)
+		(pin "47"
+		)
+		(pin "27"
+		)
+		(pin "36"
+		)
+		(pin "39"
+		)
+		(pin "38"
+		)
+		(pin "59"
+		)
+		(pin "65"
+		)
+		(pin "33"
+		)
+		(pin "37"
+		)
+		(pin "57"
+		)
+		(pin "60"
+		)
+		(pin "24"
+		)
+		(pin "44"
+		)
+		(pin "28"
+		)
+		(pin "43"
+		)
+		(pin "54"
+		)
+		(pin "49"
+		)
+		(pin "30"
+		)
+		(pin "40"
+		)
+		(pin "29"
+		)
+		(pin "31"
+		)
+		(pin "48"
+		)
+		(pin "35"
+		)
+		(pin "52"
+		)
+		(pin "41"
+		)
+		(pin "34"
+		)
+		(instances
+			(project ""
+				(path "/a1548337-1355-40e9-bc99-5140aa8d75a0"
+					(reference "U1")
+					(unit 1)
+				)
+			)
+		)
+	)
 	(sheet_instances
 		(path "/"

Commit message: last test for the git ignore
Parts:
- added C1: C, symbol Device:C
- added R1: R_Small, symbol Device:R_Small
- added SW1: SW_Push, symbol Switch:SW_Push
Connections:
- new net: C1.1, SW1.2
Other:
- moved on the sheet: U1
Changed lines of the file:
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@@
 	(paper "A4")
 	(symbol
+		(lib_id "Device:R_Small")
+		(at 78.74 45.72 0)
+		(unit 1)
+		(exclude_from_sim no)
+		(in_bom yes)
+		(on_board yes)
+		(dnp no)
+		(fields_autoplaced yes)
+		(property "Reference" "R1"
+			(at 81.28 44.4499 0)
+			(effects
+				(font
+					(size 1.016 1.016)
+				)
+				(justify left)
+			)
+		)
+		(property "Value" "R_Small"
+			(at 81.28 46.9899 0)
+			(effects
+				(font
+					(size 1.27 1.27)
+				)
+				(justify left)
+			)
+		)
+		(property "Footprint" ""
+			(at 78.74 45.72 0)
+			(effects
+				(font
+					(size 1.27 1.27)
+				)
+				(hide yes)
+			)
+		)
+		(property "Datasheet" "~"
+			(at 78.74 45.72 0)
+			(effects
+				(font
+					(size 1.27 1.27)
+				)
+				(hide yes)
+			)
+		)
+		(property "Description" "Resistor, small symbol"
+			(at 78.74 45.72 0)
+			(effects
+				(font
+					(size 1.27 1.27)
+				)
+				(hide yes)
+			)
+		)
+		(pin "1"
+		)
+		(pin "2"
+		)
+		(instances
+			(project ""
+				(path "/a1548337-1355-40e9-bc99-5140aa8d75a0"
+					(reference "R1")
+					(unit 1)
+				)
+			)
+		)
+	)
+	(symbol
 		(lib_id "RF_Module:ESP32-S3-MINI-1U")
-		(at 100.33 54.61 0)
+		(at 151.13 73.66 0)
 		(unit 1)
 		(exclude_from_sim no)
@@
 		(fields_autoplaced yes)
 		(property "Reference" "U1"
-			(at 102.4733 21.59 0)
+			(at 153.2733 40.64 0)
 			(effects
 				(font
@@
 		)
 		(property "Value" "ESP32-S3-MINI-1U"
-			(at 102.4733 24.13 0)
+			(at 153.2733 43.18 0)
 			(effects
 				(font
@@
 		)
 		(property "Footprint" "RF_Module:ESP32-S2-MINI-1U"
-			(at 116.84 83.82 0)
+			(at 167.64 102.87 0)
 			(effects
 				(font
@@
 		)
 		(property "Datasheet" "https://www.espressif.com/sites/default/files/documentation/esp32-s3-mini-1_mini-1u_datasheet_en.pdf"
-			(at 100.33 13.97 0)
+			(at 151.13 33.02 0)
 			(effects
 				(font
@@
 		)
 		(property "Description" "RF Module, ESP32-S3 SoC, Wi-Fi 802.11b/g/n, Bluetooth, BLE, 32-bit, 3.3V, SMD, external antenna"
-			(at 100.33 11.43 0)
+			(at 151.13 30.48 0)
 			(effects
 				(font
@@
 					(unit 1)
 				)
+			)
+		)
+	)
+	(symbol
+		(lib_id "Device:C")
+		(at 76.2 53.34 0)
+		(unit 1)
+		(exclude_from_sim no)
+		(in_bom yes)
+		(on_board yes)
+		(dnp no)
+		(fields_autoplaced yes)
+		(property "Reference" "C1"
+			(at 80.01 52.0699 0)
+			(effects
+				(font
+					(size 1.27 1.27)
+				)
+				(justify left)
+			)
+		)
+		(property "Value" "C"
+			(at 80.01 54.6099 0)
+			(effects
+				(font
+					(size 1.27 1.27)
+				)
+				(justify left)
+			)
+		)
+		(property "Footprint" ""
+			(at 77.1652 57.15 0)
+			(effects
+				(font
+					(size 1.27 1.27)
+				)
+				(hide yes)
+			)
+		)
+		(property "Datasheet" "~"
+			(at 76.2 53.34 0)
+			(effects
+				(font
+					(size 1.27 1.27)
+				)
+				(hide yes)
+			)
+		)
+		(property "Description" "Unpolarized capacitor"
+			(at 76.2 53.34 0)
+			(effects
+				(font
+					(size 1.27 1.27)
+				)
+				(hide yes)
+			)
+		)
+		(pin "1"
+		)
+		(pin "2"
+		)
+		(instances
+			(project ""
+				(path "/a1548337-1355-40e9-bc99-5140aa8d75a0"
+					(reference "C1")
+					(unit 1)
+				)
+			)
+		)
+	)
+	(symbol
+		(lib_id "Switch:SW_Push")
+		(at 71.12 49.53 0)
+		(unit 1)
+		(exclude_from_sim no)
+		(in_bom yes)
+		(on_board yes)
+		(dnp no)
+		(fields_autoplaced yes)
+		(property "Reference" "SW1"
+			(at 71.12 41.91 0)
+			(effects
+				(font
+					(size 1.27 1.27)
+				)
+			)
+		)
+		(property "Value" "SW_Push"
+			(at 71.12 44.45 0)
+			(effects
+				(font
+					(size 1.27 1.27)
+				)
+			)
+		)
+		(property "Footprint" ""
+			(at 71.12 44.45 0)
+			(effects
+				(font
+					(size 1.27 1.27)
+				)
+				(hide yes)
+			)
+		)
+		(property "Datasheet" "~"
+			(at 71.12 44.45 0)
+			(effects
+				(font
+					(size 1.27 1.27)
+				)
+				(hide yes)
+			)
+		)
+		(property "Description" "Push button switch, generic, two pins"
+			(at 71.12 49.53 0)
+			(effects
+				(font
+					(size 1.27 1.27)
+				)
+				(hide yes)
+			)
+		)
+		(pin "1"
+		)
+		(pin "2"
+		)
+		(instances
+			(project ""
+				(path "/a1548337-1355-40e9-bc99-5140aa8d75a0"
+					(reference "SW1")
+					(unit 1)
+				)

Commit message: buck converter implementation
Other:
- added sheet SistemaDeAlimentacion (SistemaDeAlimentacion.kicad_sch)
Changed lines of the file:
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@@
+		)
+	)
+	(sheet
+		(at 50.8 82.55)
+		(size 38.1 26.67)
+		(exclude_from_sim no)
+		(in_bom yes)
+		(on_board yes)
+		(dnp no)
+		(fields_autoplaced yes)
+		(stroke
+			(width 0.1524)
+			(type solid)
+		)
+		(fill
+			(color 0 0 0 0.0000)
+		)
+		(property "Sheetname" "SistemaDeAlimentacion"
+			(at 50.8 81.8384 0)
+			(effects
+				(font
+					(size 1.27 1.27)
+				)
+				(justify left bottom)
+			)
+		)
+		(property "Sheetfile" "SistemaDeAlimentacion.kicad_sch"
+			(at 50.8 109.8046 0)
+			(effects
+				(font
+					(size 1.27 1.27)
+				)
+				(justify left top)
+			)
+		)
+		(instances
+			(project "CanSatPCB"
+				(path "/a1548337-1355-40e9-bc99-5140aa8d75a0"
+					(page "2")
+				)
+			)
 		)
 	)
